File: VCF/VCF.kicad_pcb (KiCad board)
At the start: 2 copper layers, 136.8 x 128.5 mm, 79 parts, among them J1 AUDIO_IN, J2 CV1, J3 CV2, J4 AUDIO_OUT, J5 Conn_02x05_Odd_Even, J6 Conn_01x05_Male, J7 Conn_01x05_Female, J8 Conn_01x08_Male, J9 Conn_01x08_Female, SW1 SW_DPDT_x2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

Commit message: Updated PCBs
Parts:
- moved REF** 9.12 mm to (63.5, 54.5)
- moved REF** 9.12 mm to (73.6, 142.5)
- moved REF** 9.12 mm to (73.6, 123.0)
- moved REF** 9.12 mm to (53.4, 123.0)
- moved REF** 9.12 mm to (73.6, 69.5)
- moved REF** 9.12 mm to (53.4, 142.5)
- moved REF** 9.12 mm to (73.6, 84.0)
- moved REF** 9.12 mm to (53.4, 103.5)
- moved REF** 9.12 mm to (53.4, 84.0)
- moved REF** 9.12 mm to (50.9, 156.2)
- moved REF** 9.12 mm to (73.6, 103.5)
- moved REF** 9.12 mm to (50.9, 33.8)
- moved Ref** 9.12 mm to (73.9, 156.5)
Other:
- board size 136.8 x 128.5 mm -> 145.9 x 128.5 mm
