File: VCF/KiCad Files/VCF.kicad_pcb (KiCad board)
At the start: 2 copper layers, 156.1 x 128.5 mm, 79 parts, among them J1 CV1, J2 CV2, J3 AUDIO_IN, J4 AUDIO_OUT, J5 Conn_02x05_Odd_Even, J6 Conn_01x05_Male, J7 Conn_01x05_Female, J8 Conn_01x08_Male, J9 Conn_01x08_Female, SW1 SW_DPDT_x2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

Commit message: Update VCF.kicad_pcb
Routing:
- added copper zone on B.Cu, net (none)
- added copper zone on F.Cu, net (none)
Changed lines of the file:
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@@
   (segment (start 120.57452 78.085237) (end 116.688803 74.199519) (width 0.25) (layer "F.Cu") (net 51))
   (segment (start 120.57452 88.678084) (end 120.57452 78.085237) (width 0.25) (layer "F.Cu") (net 51))
+  (zone (net 0) (net_name "") (layer "F.Cu") (hatch edge 0.508)
+    (connect_pads (clearance 0.254))
+    (min_thickness 0.254) (filled_areas_thickness no)
+    (fill yes (thermal_gap 0.254) (thermal_bridge_width 0.254))
+    (polygon
+      (pts
+        (xy 140.75 150.5)
+        (xy 99.5 150.5)
+        (xy 99.5 39.5)
+        (xy 140.75 39.5)
+      )
+    )
+  )
   (zone (net 9) (net_name "GND") (layer "F.Cu") (hatch edge 0.508)
     (connect_pads (clearance 0.254))
@@
       )
     )
+  )
+  (zone (net 0) (net_name "") (layer "B.Cu") (hatch edge 0.508)
+    (connect_pads (clearance 0.254))
+    (min_thickness 0.254) (filled_areas_thickness no)
+    (fill yes (thermal_gap 0.254) (thermal_bridge_width 0.254))
+    (polygon
+      (pts
+        (xy 199.875 139.5)
+        (xy 158.625 139.5)
+        (xy 158.625 46.75)
+        (xy 199.875 46.75)
+      )
+    )
